Commit message: Added camera

File: urdf/robot_tutorial.xacro (robot description, xacro)
@@ -10,5 +10,6 @@
   <xacro:property name="caster_wheel_mass" value="0.001"/>
   <xacro:property name="caster_wheel_joint_offset" value="-0.052"/>
-  <!--Color Properties-->
+  <xacro:property name="camera_link_size" value="0.025" />
+  <!--Color Properties -->
   <material name="blue">
     <color rgba="0 0 0.8 1"/>
@@ -23,5 +24,5 @@
     <color rgba="0.8 0.0 0.0 1.0"/>
   </material>
-  <!--Interial macros-->
+  <!--Interial macros -->
   <xacro:macro name="cylinder_inertia" params="m r h">
     <inertial>
@@ -42,5 +43,5 @@
     </inertial>
   </xacro:macro>
-  <!--Base Footprint-->
+  <!--Base Footprint -->
   <link name="base_footprint">
     <xacro:box_inertia m="10" w="0.001" h="0.001" d="0.001"/>
@@ -52,5 +53,5 @@
     </visual>
   </link>
-  <!--Base link-->
+  <!--Base link -->
   <link name="base_link">
     <xacro:box_inertia m="10" w="${base_len}" h="${base_width}" d="0.01"/>
@@ -67,5 +68,5 @@
     </collision>
   </link>
-  <!--base_link to base_footprint Joint-->
+  <!--base_link to base_footprint Joint -->
   <joint name="base_link_joint" type="fixed">
     <origin xyz="0 0 ${wheel_radius + 0.005}" rpy="0 0 0" />
@@ -73,5 +74,5 @@
     <child link="base_link" />
   </joint>
-  <!--Wheel link & joint macro-->
+  <!--Wheel link & joint macro -->
   <xacro:macro name="wheel" params="prefix reflect">
     <link name="${prefix}_wheel">
@@ -98,8 +99,8 @@
     </joint>
   </xacro:macro>
-  <!--Create Left & Right Wheel links/joints-->
+  <!--Create Left & Right Wheel links/joints -->
   <xacro:wheel prefix="left" reflect="1"/>
   <xacro:wheel prefix="right" reflect="-1"/>
-  <!--Caster Wheel Link-->
+  <!--Caster Wheel Link -->
   <link name="caster_wheel">
     <visual>
@@ -118,5 +119,5 @@
     <xacro:sphere_inertia m="10" r="${caster_wheel_radius}"/>
   </link>
-  <!--Caster Wheel Joint-->
+  <!--Caster Wheel Joint -->
   <joint name="caster_wheel_joint" type="continuous">
     <axis xyz="0 1 0" rpy="0 0 0" />
@@ -125,4 +126,28 @@
     <origin xyz="${caster_wheel_joint_offset} 0 -${caster_wheel_radius+0.005}" rpy="0 0 0"/>
   </joint>
+  <!-- Camera link -->
+  <link name="camera_link">
+    <visual>
+      <origin xyz="0 0 0" rpy="0 0 0"/>
+      <geometry>
+        <box size="${camera_link_size} ${camera_link_size} ${camera_link_size}"/>
+      </geometry>
+      <material name="white"/>
+    </visual>
+    <collision>
+      <origin xyz="0 0 0" rpy="0 0 0"/>
+      <geometry>
+        <box size="${camera_link_size} ${camera_link_size} ${camera_link_size}"/>
+      </geometry>
+    </collision>
+    <xacro:box_inertia m="1" w="${camera_link_size}" h="${camera_link_size}" d="${camera_link_size}"/>
+  </link>
+  <!-- Camera Joint -->
+  <joint name="camera_joint" type="fixed">
+    <axis xyz="0 1 0" />
+    <origin xyz="${0.5*base_len - 0.5*camera_link_size} 0 ${0.5*camera_link_size + 0.005}" rpy="0 0 0"/>
+    <parent link="base_link"/>
+    <child link="camera_link"/>
+  </joint>
   <xacro:include filename="$(find ros_tutorial)/urdf/robot_tutorial_gazebo.xacro"/>
 </robot>

File: urdf/robot_tutorial_gazebo.xacro (robot description, xacro)
@@ -17,3 +17,43 @@
     </plugin>
   </gazebo>
+  <!-- camera -->
+  <gazebo reference="camera_link">
+    <sensor type="camera" name="camera1">
+      <update_rate>30.0</update_rate>
+      <camera name="head">
+        <horizontal_fov>1.3962634</horizontal_fov>
+        <image>
+          <width>800</width>
+          <height>800</height>
+          <format>R8G8B8</format>
+        </image>
+        <clip>
+          <near>0.02</near>
+          <far>300</far>
+        </clip>
+        <noise>
+          <type>gaussian</type>
+          <!-- Noise is sampled independently per pixel on each frame.
+               That pixel's noise value is added to each of its color
+               channels, which at that point lie in the range [0,1]. -->
+          <mean>0.0</mean>
+          <stddev>0.007</stddev>
+        </noise>
+      </camera>
+      <plugin name="camera_controller" filename="libgazebo_ros_camera.so">
+        <alwaysOn>true</alwaysOn>
+        <updateRate>0.0</updateRate>
+        <cameraName>robot_camera</cameraName>
+        <imageTopicName>image_raw</imageTopicName>
+        <cameraInfoTopicName>camera_info</cameraInfoTopicName>
+        <frameName>camera_link</frameName>
+        <hackBaseline>0.07</hackBaseline>
+        <distortionK1>0.0</distortionK1>
+        <distortionK2>0.0</distortionK2>
+        <distortionK3>0.0</distortionK3>
+        <distortionT1>0.0</distortionT1>
+        <distortionT2>0.0</distortionT2>
+      </plugin>
+    </sensor>
+  </gazebo>
 </robot>

Commit message: Added 360 lidar, but still only inf right now...

File: urdf/robot_tutorial.xacro (robot description, xacro)
@@ -10,4 +10,7 @@
   <xacro:property name="caster_wheel_mass" value="0.001"/>
   <xacro:property name="caster_wheel_joint_offset" value="-0.052"/>
+  <xacro:property name="lidar360_link_height" value="0.075" />
+  <xacro:property name="lidar360_link_size" value="0.025" />
+  <xacro:property name="lidar360_dist" value="0.025" /> <!-- Distance above mount for lidar frame-->
   <!--Color Properties-->
   <material name="blue">
@@ -125,4 +128,35 @@
     <origin xyz="${caster_wheel_joint_offset} 0 -${caster_wheel_radius+0.005}" rpy="0 0 0"/>
   </joint>
+  <!-- Lidar360 Links-->
+  <link name="lidar360_link">
+    <visual>
+      <origin xyz="0 0 0" rpy="0 0 0"/>
+      <geometry>
+        <box size="${lidar360_link_size} ${lidar360_link_size} ${lidar360_link_height}"/>
+      </geometry>
+      <material name="white"/>
+    </visual>
+    <collision>
+      <origin xyz="0 0 0" rpy="0 0 0"/>
+      <geometry>
+        <box size="${lidar360_link_size} ${lidar360_link_size} ${lidar360_link_height}"/>
+      </geometry>
+    </collision>
+    <xacro:box_inertia m="2" w="${lidar360_link_size}" h="${lidar360_link_height}" d="${lidar360_link_size}"/>
+  </link>
+  <link name="laser" />
+  <!-- Lidar360 Joints-->
+  <joint name="lidar360_joint" type="fixed">
+    <axis xyz="0 1 0" />
+    <origin xyz="${-0.5*base_len + 0.5*lidar360_link_size} 0 ${0.5*lidar360_link_height + 0.005}" rpy="0 0 0"/>
+    <parent link="base_link"/>
+    <child link="lidar360_link"/>
+  </joint>
+  <joint name="lidar360_top_joint" type="fixed">
+    <axis xyz="0 1 0" />
+    <origin xyz="0 0 ${0.5*lidar360_link_height + 0.5*lidar360_dist}" rpy="0 0 0"/>
+    <parent link="lidar360_link"/>
+    <child link="laser"/>
+  </joint>
   <xacro:include filename="$(find ros_tutorial)/urdf/robot_tutorial_gazebo.xacro"/>
 </robot>

File: urdf/robot_tutorial_gazebo.xacro (robot description, xacro)
@@ -17,3 +17,38 @@
     </plugin>
   </gazebo>
+  <gazebo reference="laser">
+    <sensor type="gpu_ray" name="laser">
+      <pose>0 0 0 0 0 0</pose>
+      <visualize>false</visualize>
+      <update_rate>40</update_rate>
+      <ray>
+        <scan>
+          <horizontal>
+            <samples>720</samples>
+            <resolution>1</resolution>
+            <min_angle>-1.570796</min_angle>
+            <max_angle>1.570796</max_angle>
+          </horizontal>
+        </scan>
+        <range>
+          <min>0.1</min>
+          <max>30.0</max>
+          <resolution>0.01</resolution>
+        </range>
+        <noise>
+          <type>gaussian</type>
+          <!-- Noise parameters based on published spec for Hokuyo laser
+               achieving "+-30mm" accuracy at range < 10m.  A mean of 0.0m and
+               stddev of 0.01m will put 99.7% of samples within 0.03m of the true
+               reading. -->
+          <mean>0.0</mean>
+          <stddev>0.01</stddev>
+        </noise>
+      </ray>
+      <plugin name="gazebo_ros_head_hokuyo_controller" filename="libgazebo_ros_gpu_laser.so">
+        <topicName>scan</topicName>
+        <frameName>laser</frameName>
+      </plugin>
+    </sensor>
+  </gazebo>
 </robot>
